Commit message: update model

File: src/mybot_description/urdf/mybot.xacro (robot description, xacro)
@@ -9,5 +9,5 @@
     <pose>0 0 0.1 0 0 0</pose>
     <inertial>
-      <mass value="10.0"/>
+      <mass value="15.0"/>
       <origin xyz="0.0 0 0.1" rpy=" 0 0 0"/>
       <inertia
@@ -142,5 +142,5 @@
     <child link="camera"/>
   </joint>
-  <joint name="hokuyo_joint" type="fixed">
+  <!-- <joint name="hokuyo_joint" type="fixed">
     <axis xyz="0 1 0" />
     <origin xyz=".15 0 .1" rpy="0 0 0"/>
@@ -148,5 +148,4 @@
     <child link="hokuyo"/>
   </joint>
-  <!-- Hokuyo Laser -->
   <link name="hokuyo">
     <collision>
@@ -167,4 +166,4 @@
       <inertia ixx="1e-6" ixy="0" ixz="0" iyy="1e-6" iyz="0" izz="1e-6" />
     </inertial>
-  </link>
+  </link> -->
 </robot>
